Commit message: make the rover usable in Gazebo
Hooked up diff drive and joint states, then added simulated lidar/IMU
sensors. The bridge carries cmd_vel, odom, scan, TF, and the remaining
sensor topics back into ROS 2.

File: src/rover_description/urdf/rover.urdf.xacro (robot description, xacro)
@@ -48,3 +48,27 @@
     <parent link="base_link"/><child link="imu_link"/><origin xyz="0 0 0.06"/>
   </joint>
+  <gazebo reference="base_link"><material>Gazebo/Green</material></gazebo>
+  <gazebo reference="left_wheel_link"><mu1>1.0</mu1><mu2>1.0</mu2></gazebo>
+  <gazebo reference="right_wheel_link"><mu1>1.0</mu1><mu2>1.0</mu2></gazebo>
+  <gazebo>
+    <plugin filename="gz-sim-diff-drive-system" name="gz::sim::systems::DiffDrive">
+      <left_joint>left_wheel_joint</left_joint>
+      <right_joint>right_wheel_joint</right_joint>
+      <wheel_separation>${2 * wheel_y}</wheel_separation>
+      <wheel_radius>${wheel_radius}</wheel_radius>
+      <topic>cmd_vel</topic><odom_topic>odom</odom_topic><frame_id>odom</frame_id><child_frame_id>base_footprint</child_frame_id>
+    </plugin>
+    <plugin filename="gz-sim-joint-state-publisher-system" name="gz::sim::systems::JointStatePublisher"/>
+  </gazebo>
+  <gazebo reference="lidar_link">
+    <sensor name="lidar" type="gpu_lidar">
+      <topic>scan</topic><update_rate>10</update_rate><always_on>true</always_on><visualize>true</visualize>
+      <lidar><scan><horizontal><samples>720</samples><resolution>1</resolution><min_angle>-3.14159</min_angle><max_angle>3.14159</max_angle></horizontal></scan>
+        <range><min>0.12</min><max>12.0</max><resolution>0.01</resolution></range>
+      </lidar>
+    </sensor>
+  </gazebo>
+  <gazebo reference="imu_link">
+    <sensor name="imu" type="imu"><topic>imu/data</topic><update_rate>50</update_rate><always_on>true</always_on></sensor>
+  </gazebo>
 </robot>
